Commit message: urdf with laser and kinect

File: urdf/standford_pupper.urdf (robot description, URDF)
Before this commit: robot stanford_pupper, 18 links, 17 joints
Links:
- added link camera_depth_frame
- added link camera_depth_optical_frame
- added link camera_link, mass 0.200; collision mesh filename=package://hector_sensors_description/meshes/asus_camera/asu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; visual mesh filename=package://hector_sensors_description/meshes/asus_camera/asu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
- added link camera_rgb_frame
- added link camera_rgb_optical_frame
- added link hokuyo_frame, mass 0.270; collision box size=0.058 0.058 0.087; visual mesh filename=package://hector_sensors_description/meshes/hokuyo_utm30lx/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
Joints:
- added joint camera_depth_joint: type fixed, parent camera_link, child camera_depth_frame, origin xyz=0.0 0.049 0.0 rpy=0 0 0
- added joint camera_depth_optical_joint: type fixed, parent camera_depth_frame, child camera_depth_optical_frame, origin xyz=0 0 0 rpy=-1.5707963267948966 0.0 -1.5707963267948966
- added joint camera_joint: type fixed, parent base_link, child camera_link, origin xyz=0.098 0.0 0.082 rpy=0 0 0
- added joint camera_rgb_joint: type fixed, parent camera_link, child camera_rgb_frame, origin xyz=0.0 0.022 0.0 rpy=0 0 0
- added joint camera_rgb_optical_joint: type fixed, parent camera_rgb_frame, child camera_rgb_optical_frame, origin xyz=0 0 0 rpy=-1.5707963267948966 0.0 -1.5707963267948966
- added joint hokuyo_joint: type fixed, parent base_link, child hokuyo_frame, origin xyz=-0.05 0.0 0.1 rpy=0 0 0
